Commit message: tune(demo): firmer/gentler finger grip + contact diagnostics (genuine grasp WIP)
Toward a genuine (physics-only) friction grasp:
- Raise finger effort limit 20 -> 150 N and add a position PID (p=1500, d=5) so
  closing applies a real squeeze force.
- Slow the finger close velocity 0.2 -> 0.04 m/s so contact builds symmetrically
  instead of slamming the object out of the gripper.
- Driver logs the finger opening after the squeeze (contact diagnostic).

Characterized failure modes (gz/DART friction grasping is the known-hard part):
weak grip -> object rises ~8mm then slips; firm+fast grip -> fingers eject the
free object and close to 0; position-controlled gripper can't hold a constant
force. Geometry/targeting is correct (fingers reach the object, stall on it).
Next lever: an EFFORT (force) command interface on the fingers, not position.

File: ros2_ws/src/generated_objects_eval/urdf/panda_base.urdf (robot description, URDF)
Before this commit: robot panda, 12 links, 11 joints
Joints:
- joint panda_finger_joint1: limit lower=0.0 upper=0.04 effort=20 velocity=0.2 -> lower=0.0 upper=0.04 effort=150 velocity=0.04
- joint panda_finger_joint2: limit lower=0.0 upper=0.04 effort=20 velocity=0.2 -> lower=0.0 upper=0.04 effort=150 velocity=0.04
